File: FM_Receiver/FM_Receiver.kicad_sch (KiCad schematic)
At the start: 27 parts, among them J1 USB_C_Receptacle_PowerOnly_6P, U1 LM380N-8, U2 LM380N-8, U3 Si4731-D60-GU, U4 FUSB302B01MPX

Commit message: new updates
Dec. 3 update
Parts:
- removed C10, C8: 1000uF_50V, Capacitor_SMD:C_0201_0603Metric, symbol PCM_SL_Capacitors:22uF_50V
- removed R3, R4: 10, Resistor_SMD:R_0201_0603Metric_Pad0.64x0.40mm_HandSolder, symbol PCM_Elektuur:R
- added C8: 500µ, Capacitor_SMD:C_0201_0603Metric, symbol PCM_Elektuur:C
- added R5, R6: 5K, Resistor_SMD:R_0201_0603Metric_Pad0.64x0.40mm_HandSolder, symbol PCM_Elektuur:R
- A1: footprint PCM_arduino-library:Arduino_Uno_R4_WiFi_Shield -> DigiKey_ABX00087:ARDUINO UNO R4 WIFI_ABX00087
- C11, C12, C13, C3, C5, C6, C7: footprint Capacitor_SMD:C_0201_0603Metric -> Capacitor_THT:CP_Radial_D5.0mm_P2.00mm
- C14: footprint Capacitor_SMD:C_0201_0603Metric -> Capacitor_THT:CP_Radial_D5.0mm_P2.50mm
- C2: value 1nF -> 500µ
- R1, R2: footprint Resistor_SMD:R_0201_0603Metric_Pad0.64x0.40mm_HandSolder -> Resistor_THT:R_Axial_DIN0207_L6.3mm_D2.5mm_P10.16mm_Horizontal
- U4: footprint Package_DFN_QFN:WQFN-14-1EP_2.5x2.5mm_P0.5mm_EP1.45x1.45mm_ThermalVias -> Package_DFN_QFN:WQFN-14-1EP_2.5x2.5mm_P0.5mm_EP1.45x1.45mm
Connections:
- net +20V is gone; now on net +12V: U2.7 (VS)
- net +3.3V: now also U4.12 (VCONN), U4.13 (VCONN), R5.1 (+), R6.1 (+)
- net at C12.1, U1.6: now also C2.1 (+)
- net at LS1.1: now also C2.2 (-)
- net at FM_ANTENNA1.1 (A): now also U3.8 (FMI); no longer C2.1 (+)
- net at RS1.1: now also C8.2 (-)
- net at C13.1, U2.6: now also C8.1 (+)
- net at A1.SCL, U4.6 (SCL): now also R6.2 (-)
- net at A1.SDA, U4.7 (SDA): now also R5.2 (-)
Other:
- company: (none) -> Self - Bertin Mihigo Sano
- title: (none) -> FM Radio Digital Analog
- moved on the sheet: A1, C1, C11, C12, C13, C14, C3, C4, C5, C6, C7, C9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
